File: circ/Flaptastic_595_kicad/Flaptastic_595/Flaptastic_595.kicad_pcb (KiCad board)
At the start: 2 copper layers, 62.2 x 35.6 mm, 18 parts, among them J1 IN, J2 OUT, J3 Stepper logic, J4 Stepper power, J5 Stepper power, J6 Stepper power, Q1 IR Phototransistor, Q2 PN2222A, U1 74HC595

Commit message: Worked on PCB, rm bak files
Parts:
- added J7: Digital outputs, Connector_PinHeader_2.54mm:PinHeader_1x02_P2.54mm_Vertical, F.Cu at (125.7, 134.6)
- added JP3: Stepper +V feed, Jumper:SolderJumper-2_P1.3mm_Open_RoundedPad1.0x1.5mm, B.Cu at (93.3, 137.8)
- added JP4: Stepper GND feed, Jumper:SolderJumper-2_P1.3mm_Open_RoundedPad1.0x1.5mm, B.Cu at (93.3, 134.0)
- JP1: value CE bypass -> CLK bypass; moved to B.Cu
- JP2: moved to B.Cu
- moved JP1 11.4 mm to (115.6, 135.3)
- moved J3 7.62 mm to (86.4, 116.8), turned to 180 degrees
- moved JP2 7.10 mm to (90.2, 122.6), turned to 270 degrees
- moved D1 2.54 mm to (132.1, 129.5), turned to 0 degrees
- moved J6 1.31 mm to (81.4, 119.4)
Connections:
- C2 pad 1: /CE -> VCC
- J1 pad 1: /CLK_IN -> /RETURN
- J1 pad 10: Earth -> /STEPPER_GND_IN
- J1 pad 2: /SER_IN -> /CLK_IN
- J1 pad 5: /RETURN -> /nOE
- J1 pad 6: /CE -> /SER_IN
- J1 pad 7: /nOE -> /STEPPER_V_IN
- J1 pad 8: +5V -> /STEPPER_V_IN
- J1 pad 9: Earth -> /STEPPER_GND_IN
- J2 pad 1: (no net) -> /RETURN
- J2 pad 10: (no net) -> Earth
- J2 pad 2: (no net) -> /CLK
- J2 pad 3: (no net) -> VCC
- J2 pad 4: (no net) -> GND
- J2 pad 5: (no net) -> /nOE
- J2 pad 6: (no net) -> /SER_OUT
- J2 pad 7: (no net) -> +5V
- J2 pad 8: (no net) -> +5V
- J2 pad 9: (no net) -> Earth
- JP2 pad 1: /D2\SER_OUT -> /SER_OUT
- Q2 pad 3: /CE -> VCC
- R1 pad 1: /D2\SER_OUT -> /SER_OUT
- U1 pad 1: /M0 -> /D0
- U1 pad 15: (no net) -> /D1
- U1 pad 2: /M1 -> /M3
- U1 pad 4: /M3 -> /M1
- U1 pad 5: (no net) -> /M0
- U1 pad 6: /D2\SER_OUT -> /SER_OUT
Routing:
- net /SER_OUT: track 0.00 -> 59.7 mm, vias 0 -> 1
- net /D2\SER_OUT: track 40.3 -> 0.00 mm
- net /RETURN: track 18.8 -> 55.4 mm, vias 0 -> 1
- net /D1: track 0.00 -> 32.7 mm, vias 0 -> 1
- net VCC: track 61.4 -> 93.0 mm, vias 0 -> 1
- net /CE: track 30.8 -> 0.00 mm
- net /D0: track 0.00 -> 30.2 mm, vias 0 -> 1
- net Earth: track 69.2 -> 97.8 mm, vias 1 -> 3
- net +5V: track 82.1 -> 102.8 mm, vias 0 -> 1
- net /nOE: track 9.20 -> 27.5 mm
- net /CLK: track 42.3 -> 59.7 mm
- net GND: track 69.4 -> 83.8 mm, vias 1 -> 2
- net /M0: track 30.2 -> 16.3 mm
- net /STEPPER_V_IN: track 0.00 -> 10.9 mm
- net /CLK_IN: track 21.1 -> 12.0 mm
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Other:
- net class Default: clearance 0.2 -> 0.1524; trace_width 0.25 -> 0.1524; via_dia 0.8 -> 0.8128; via_drill 0.4 -> 0.4064
- rule pad_to_mask_clearance: 0.051 -> 0.0508
- rule solder_mask_min_width: 0.25 -> 0.1016
- rule trace_clearance: 0.2 -> 0.1524
- rule trace_min: 0.2 -> 0.1524
- rule via_min_drill: 0.3 -> 0.254
- rule via_min_size: 0.4 -> 0.508
