File: circ/Flaptastic_595_kicad/Flaptastic_595/Flaptastic_595.sch (KiCad schematic (older format))
At the start: 18 parts, among them J1 IN, J2 OUT, J3 Stepper logic, J4 Stepper power, J5 Stepper power, J6 Stepper power, Q1 IR Phototransistor, Q2 PN2222A, U1 74HC595

Commit message: Worked on PCB, rm bak files
Parts:
- added J7: Digital outputs, Connector_PinHeader_2.54mm:PinHeader_1x02_P2.54mm_Vertical, symbol Connector_Generic:Conn_01x02
- added JP3: Stepper +V feed, Jumper:SolderJumper-2_P1.3mm_Open_RoundedPad1.0x1.5mm, symbol Jumper:SolderJumper_2_Open
- added JP4: Stepper GND feed, Jumper:SolderJumper-2_P1.3mm_Open_RoundedPad1.0x1.5mm, symbol Jumper:SolderJumper_2_Open
- JP1: value CE bypass -> CLK bypass
Connections:
- net D2\SER_OUT is gone; now on net SER_OUT: JP2.1 (A), R1.1, U1.6 (QG)
- net +5V: now also J2.7 (Pin_7), J2.8 (Pin_8), JP3.2 (B); no longer J1.8 (Pin_8)
- net CLK: now also J2.2 (Pin_2)
- net CLK_IN: now also J1.2 (Pin_2); no longer J1.1 (Pin_1)
- net D0: now also U1.1 (QB), J7.1 (Pin_1); no longer U1.15 (QA)
- net D1: now also U1.15 (QA), J7.2 (Pin_2); no longer U1.5 (QF)
- net Earth: now also J2.10 (Pin_10), J2.9 (Pin_9), JP4.2 (B); no longer J1.10 (Pin_10), J1.9 (Pin_9)
- net GND: now also J2.4 (Pin_4)
- net M0: now also U1.5 (QF); no longer U1.1 (QB)
- net M1: now also U1.4 (QE); no longer U1.2 (QC)
- net M3: now also U1.2 (QC); no longer U1.4 (QE)
- net RETURN: now also J1.1 (Pin_1), J2.1 (Pin_1); no longer J1.5 (Pin_5)
- net SER_IN: now also J1.6 (Pin_6); no longer J1.2 (Pin_2)
- net VCC: now also C2.1, J2.3 (Pin_3), Q2.3 (C)
- net nOE: now also J1.5 (Pin_5), J2.5 (Pin_5); no longer J1.7 (Pin_7)
- net SER_OUT: now reaches J2.6 (Pin_6)
- removed net CE: C2.1, J1.6 (Pin_6), Q2.3 (C)
- net D3: no longer names the net of U1.7 (QH)
- new net STEPPER_GND_IN: J1.10 (Pin_10), J1.9 (Pin_9), JP4.1 (A)
- new net STEPPER_V_IN: J1.7 (Pin_7), J1.8 (Pin_8), JP3.1 (A)
- no-connect marks 7 -> 6
Other:
- moved on the sheet: J1
